Commit message: Update detector migration workspace

File: src/dobot_rviz/urdf/cr10_robot.urdf (robot description, URDF)
Before this commit: robot cr10_robot, 8 links, 7 joints
Links:
- removed link camera_link
Joints:
- removed joint camera_mount

File: src/dobot_rviz/urdf/cr12_robot.urdf (robot description, URDF)
Before this commit: robot cr12_robot, 9 links, 8 joints
Links:
- removed link camera_link
Joints:
- removed joint camera_mount

File: src/dobot_rviz/urdf/cr16_robot.urdf (robot description, URDF)
Before this commit: robot cr16_robot, 9 links, 8 joints
Links:
- removed link camera_link
Joints:
- removed joint camera_mount

File: src/dobot_rviz/urdf/cr20_robot.urdf (robot description, URDF)
Before this commit: robot cr20_robot, 9 links, 8 joints
Links:
- removed link camera_link
Joints:
- removed joint camera_mount

File: src/dobot_rviz/urdf/cr30h_robot.urdf (robot description, URDF)
Before this commit: robot cr30h_robot, 9 links, 8 joints
Links:
- removed link camera_link
Joints:
- removed joint camera_mount

File: src/dobot_rviz/urdf/cr3_robot.urdf (robot description, URDF)
Before this commit: robot cr3_robot, 9 links, 8 joints
Links:
- removed link camera_link
Joints:
- removed joint camera_mount

File: src/dobot_rviz/urdf/cr5_robot.urdf (robot description, URDF)
Before this commit: robot cr5_robot, 9 links, 8 joints
Links:
- removed link camera_link
Joints:
- removed joint camera_mount

File: src/dobot_rviz/urdf/cr7_robot.urdf (robot description, URDF)
Before this commit: robot cr7_robot, 9 links, 8 joints
Links:
- removed link camera_link
Joints:
- removed joint camera_mount

File: src/dobot_rviz/urdf/me6_robot.urdf (robot description, URDF)
Before this commit: robot me6_robot, 9 links, 8 joints
Links:
- removed link camera_link
Joints:
- removed joint camera_mount

File: src/dobot_rviz/urdf/nova2_robot.urdf (robot description, URDF)
Before this commit: robot nova2_robot, 9 links, 8 joints
Links:
- removed link camera_link
Joints:
- removed joint camera_mount

File: src/dobot_rviz/urdf/nova5_robot.urdf (robot description, URDF)
Before this commit: robot nova5_robot, 8 links, 7 joints
Links:
- removed link camera_link
Joints:
- removed joint camera_mount
